File: kicad/ard8088.kicad_pcb (KiCad board)
At the start: 2 copper layers, 104.1 x 55.9 mm, 7 parts, among them U1 8088_Max_Mode, U2 8288

Commit message: Minor updates, release PCB
Parts:
- removed R1: 4.7k, Resistor_THT:R_Axial_DIN0204_L3.6mm_D1.6mm_P5.08mm_Horizontal
- added BZ1: Buzzer, Buzzer_Beeper:Buzzer_12x9.5RM7.6, F.Cu at (165.1, 73.7)
- C2: moved to B.Cu
- moved C1 0.33 mm to (102.4, 72.3)
Connections:
- U1 pad 30: unconnected-(U1-Pad30) -> /~{RQ}/~{GT1}
- U2 pad 15: Net-(R1-Pad2) -> /CEN
- U2 pad 6: GND -> /~{AEN}
- XA1 pad A0: unconnected-(XA1-PadA0) -> /~{AEN}
- XA1 pad A1: unconnected-(XA1-PadA1) -> /CEN
- XA1 pad D3: unconnected-(XA1-PadD3) -> /~{RQ}/~{GT1}
Routing:
- net /~{RQ}/~{GT1}: track 0.00 -> 23.7 mm
- net Net-(R1-Pad2): track 22.2 -> 0.00 mm
- net unconnected-(XA1-PadD2): track 0.00 -> 21.6 mm
- net /CEN: track 0.00 -> 15.3 mm
- net /~{AEN}: track 0.00 -> 6.57 mm
- net /CLK: track 139.4 -> 140.7 mm, vias 0 -> 1
- net /S2: track 69.1 -> 70.0 mm
- net /S0: track 62.7 -> 63.4 mm
- net GND: track 16.4 -> 17.2 mm
