File: kicad/ard8088.kicad_sch (KiCad schematic)
At the start: 6 parts, among them U1 8088_Max_Mode, U2 8288

Commit message: Minor updates, release PCB
Parts:
- removed R1: 4.7k, Resistor_THT:R_Axial_DIN0204_L3.6mm_D1.6mm_P5.08mm_Horizontal, symbol Device:R
Connections:
- net GND: no longer U2.6 (~{AEN})
- net CEN: now reaches XA1.A0
- net CEN: now also U2.15 (CEN)
- net ~{AEN}: now reaches XA1.A1
- net ~{AEN}: now also U2.6 (~{AEN})
Changed lines of the file:
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@@
   (junction (at 21.59 127) (diameter 0) (color 0 0 0 0)
   )
-  (junction (at 207.01 26.67) (diameter 0) (color 0 0 0 0)
-  )
   (junction (at 161.29 26.67) (diameter 0) (color 0 0 0 0)
   )
   (junction (at 21.59 124.46) (diameter 0) (color 0 0 0 0)
-  )
-  (junction (at 201.93 90.17) (diameter 0) (color 0 0 0 0)
   )
   (junction (at 163.83 153.67) (diameter 0) (color 0 0 0 0)
@@
     (stroke (width 0) (type default) (color 0 0 0 0))
   )
+  (wire (pts (xy 199.39 85.09) (xy 209.55 85.09))
+    (stroke (width 0) (type default) (color 0 0 0 0))
+  )
   (wire (pts (xy 132.08 76.2) (xy 143.51 76.2))
     (stroke (width 0) (type default) (color 0 0 0 0))
@@
     (stroke (width 0) (type default) (color 0 0 0 0))
   )
-  (wire (pts (xy 207.01 26.67) (xy 227.33 26.67))
+  (wire (pts (xy 161.29 26.67) (xy 227.33 26.67))
     (stroke (width 0) (type default) (color 0 0 0 0))
   )
@@
     (stroke (width 0) (type default) (color 0 0 0 0))
   )
-  (wire (pts (xy 207.01 46.99) (xy 207.01 26.67))
-    (stroke (width 0) (type default) (color 0 0 0 0))
-  )
   (wire (pts (xy 130.81 134.62) (xy 143.51 134.62))
     (stroke (width 0) (type default) (color 0 0 0 0))
@@
     (stroke (width 0) (type default) (color 0 0 0 0))
   )
+  (wire (pts (xy 17.78 66.04) (xy 24.13 66.04))
+    (stroke (width 0) (type default) (color 0 0 0 0))
+  )
   (wire (pts (xy 90.17 48.26) (xy 140.97 48.26))
     (stroke (width 0) (type default) (color 0 0 0 0))
@@
     (stroke (width 0) (type default) (color 0 0 0 0))
   )
-  (wire (pts (xy 209.55 85.09) (xy 201.93 85.09))
-    (stroke (width 0) (type default) (color 0 0 0 0))
-  )
   (wire (pts (xy 21.59 127) (xy 21.59 129.54))
     (stroke (width 0) (type default) (color 0 0 0 0))
@@
     (stroke (width 0) (type default) (color 0 0 0 0))
   )
-  (wire (pts (xy 207.01 92.71) (xy 209.55 92.71))
-    (stroke (width 0) (type default) (color 0 0 0 0))
-  )
-  (wire (pts (xy 201.93 85.09) (xy 201.93 90.17))
+  (wire (pts (xy 199.39 92.71) (xy 209.55 92.71))
     (stroke (width 0) (type default) (color 0 0 0 0))
   )
@@
     (stroke (width 0) (type default) (color 0 0 0 0))
   )
+  (wire (pts (xy 17.78 68.58) (xy 24.13 68.58))
+    (stroke (width 0) (type default) (color 0 0 0 0))
+  )
   (bus (pts (xy 129.54 116.84) (xy 129.54 118.11))
     (stroke (width 0) (type default) (color 0 0 0 0))
@@
     (stroke (width 0) (type default) (color 0 0 0 0))
   )
-  (wire (pts (xy 161.29 26.67) (xy 207.01 26.67))
-    (stroke (width 0) (type default) (color 0 0 0 0))
-  )
   (wire (pts (xy 245.11 77.47) (xy 251.46 77.47))
     (stroke (width 0) (type default) (color 0 0 0 0))
@@
     (stroke (width 0) (type default) (color 0 0 0 0))
   )
-  (wire (pts (xy 207.01 54.61) (xy 207.01 92.71))
-    (stroke (width 0) (type default) (color 0 0 0 0))
-  )
   (bus (pts (xy 102.87 66.04) (xy 102.87 68.58))
     (stroke (width 0) (type default) (color 0 0 0 0))
@@
     (effects (font (size 1.27 1.27)) (justify left))
   )
+  (hierarchical_label "~{AEN}" (shape input) (at 17.78 68.58 180)
+    (effects (font (size 1.27 1.27)) (justify right))
+  )
   (hierarchical_label "DEN" (shape input) (at 251.46 95.25 0)
     (effects (font (size 1.27 1.27)) (justify left))
@@
     (effects (font (size 1.27 1.27)) (justify left))
   )
+  (hierarchical_label "CEN" (shape input) (at 199.39 92.71 180)
+    (effects (font (size 1.27 1.27)) (justify right))
+  )
   (hierarchical_label "ALE" (shape input) (at 251.46 90.17 0)
     (effects (font (size 1.27 1.27)) (justify left))
@@
     (effects (font (size 1.27 1.27)) (justify left))
   )
+  (hierarchical_label "CEN" (shape input) (at 17.78 66.04 180)
+    (effects (font (size 1.27 1.27)) (justify right))
+  )
   (hierarchical_label "DEN" (shape input) (at 93.98 119.38 0)
     (effects (font (size 1.27 1.27)) (justify left))
@@
   (hierarchical_label "INTR" (shape input) (at 184.15 81.28 0)
     (effects (font (size 1.27 1.27)) (justify left))
+  )
+  (hierarchical_label "~{AEN}" (shape input) (at 199.39 85.09 180)
+    (effects (font (size 1.27 1.27)) (justify right))
   )
   (hierarchical_label "~{MWTC}" (shape input) (at 251.46 72.39 0)
@@
     (pin "1")
   )
-  (symbol (lib_id "Device:R") (at 207.01 50.8 0) (unit 1)
-    (in_bom yes) (on_board yes) (fields_autoplaced)
-    (property "Reference" "R1" (id 0) (at 209.55 49.5299 0)
-      (effects (font (size 1.27 1.27)) (justify left))
-    )
-    (property "Value" "4.7k" (id 1) (at 209.55 52.0699 0)
-      (effects (font (size 1.27 1.27)) (justify left))
-    )
-    (property "Footprint" "Resistor_THT:R_Axial_DIN0204_L3.6mm_D1.6mm_P5.08mm_Horizontal" (id 2) (at 205.232 50.8 90)
-      (effects (font (size 1.27 1.27)) hide)
-    )
-    (property "Datasheet" "~" (id 3) (at 207.01 50.8 0)
-      (effects (font (size 1.27 1.27)) hide)
-    )
-    (pin "1")
-    (pin "2")
-  )
   (symbol (lib_id "power:+5V") (at 161.29 26.67 0) (unit 1)
     (in_bom yes) (on_board yes) (fields_autoplaced)
@@
       (reference "C2") (unit 1) (value "0.1uf") (footprint "Capacitor_SMD:C_0805_2012Metric_Pad1.18x1.45mm_HandSolder")
     )
-    (path "/6a1bb6be-af1b-4603-af6d-c401435e7f82"
-      (reference "R1") (unit 1) (value "4.7k") (footprint "Resistor_THT:R_Axial_DIN0204_L3.6mm_D1.6mm_P5.08mm_Horizontal")
-    )
     (path "/25c7c0cb-88f8-4596-a4f2-f3d27a29907e"

Commit message: Update schematic to 1.0b
Parts:
- added BZ1: Buzzer, Buzzer_Beeper:Buzzer_12x9.5RM7.6, symbol Device:Buzzer
Connections:
- net CEN: now also XA1.A1; no longer XA1.A0
- net GND: now also BZ1.2 (+)
- net ~{AEN}: now also XA1.A0; no longer XA1.A1
- net at XA1.D2 (D2_INT0): now also BZ1.1 (-)
- net ~{RQ}/~{GT1}: now reaches XA1.D3 (D3_INT1)
- net ~{RQ}/~{GT1}: now also U1.30 (~{RQ}/~{GT1})
- no-connect marks 14 -> 12
Changed lines of the file:
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@@
   (title_block
     (title "Ard8088")
-    (rev "v01")
+    (rev "v01b")
   )
   (junction (at 180.34 153.67) (diameter 0) (color 0 0 0 0)
@@
   (junction (at 163.83 153.67) (diameter 0) (color 0 0 0 0)
   )
-  (no_connect (at 90.17 35.56))
   (no_connect (at 90.17 33.02))
   (no_connect (at 179.07 129.54))
-  (no_connect (at 179.07 96.52))
   (no_connect (at 179.07 101.6))
   (no_connect (at 50.8 21.59))
@@
     (stroke (width 0) (type default) (color 0 0 0 0))
   )
+  (wire (pts (xy 90.17 33.02) (xy 93.98 33.02))
+    (stroke (width 0) (type default) (color 0 0 0 0))
+  )
   (wire (pts (xy 132.08 91.44) (xy 143.51 91.44))
     (stroke (width 0) (type default) (color 0 0 0 0))
@@
     (stroke (width 0) (type default) (color 0 0 0 0))
   )
+  (wire (pts (xy 93.98 24.13) (xy 93.98 33.02))
+    (stroke (width 0) (type default) (color 0 0 0 0))
+  )
   (wire (pts (xy 90.17 91.44) (xy 100.33 91.44))
     (stroke (width 0) (type default) (color 0 0 0 0))
@@
     (stroke (width 0) (type default) (color 0 0 0 0))
   )
+  (wire (pts (xy 90.17 35.56) (xy 104.14 35.56))
+    (stroke (width 0) (type default) (color 0 0 0 0))
+  )
   (wire (pts (xy 17.78 50.8) (xy 24.13 50.8))
     (stroke (width 0) (type default) (color 0 0 0 0))
@@
     (stroke (width 0) (type default) (color 0 0 0 0))
   )
+  (wire (pts (xy 179.07 96.52) (xy 184.15 96.52))
+    (stroke (width 0) (type default) (color 0 0 0 0))
+  )
   (wire (pts (xy 90.17 129.54) (xy 93.98 129.54))
     (stroke (width 0) (type default) (color 0 0 0 0))
@@
     (stroke (width 0) (type default) (color 0 0 0 0))
   )
+  (wire (pts (xy 99.06 24.13) (xy 99.06 29.21))
+    (stroke (width 0) (type default) (color 0 0 0 0))
+  )
   (bus (pts (xy 102.87 93.98) (xy 102.87 96.52))
     (stroke (width 0) (type default) (color 0 0 0 0))
@@
     (effects (font (size 1.27 1.27)) (justify left))
   )
-  (hierarchical_label "~{AEN}" (shape input) (at 17.78 68.58 180)
-    (effects (font (size 1.27 1.27)) (justify right))
-  )
   (hierarchical_label "DEN" (shape input) (at 251.46 95.25 0)
     (effects (font (size 1.27 1.27)) (justify left))
@@
     (effects (font (size 1.27 1.27)) (justify right))
   )
+  (hierarchical_label "~{RQ}{slash}~{GT1}" (shape input) (at 104.14 35.56 0)
+    (effects (font (size 1.27 1.27)) (justify left))
+  )
   (hierarchical_label "~{S0}" (shape input) (at 201.93 64.77 180)
     (effects (font (size 1.27 1.27)) (justify right))
@@
     (effects (font (size 1.27 1.27)) (justify left))
   )
+  (hierarchical_label "~{AEN}" (shape input) (at 17.78 66.04 180)
+    (effects (font (size 1.27 1.27)) (justify right))
+  )
   (hierarchical_label "~{MRDC}" (shape input) (at 93.98 137.16 0)
     (effects (font (size 1.27 1.27)) (justify left))
@@
     (effects (font (size 1.27 1.27)) (justify left))
   )
-  (hierarchical_label "CEN" (shape input) (at 17.78 66.04 180)
-    (effects (font (size 1.27 1.27)) (justify right))
-  )
   (hierarchical_label "DEN" (shape input) (at 93.98 119.38 0)
     (effects (font (size 1.27 1.27)) (justify left))
@@
   )
   (hierarchical_label "CLK" (shape input) (at 104.14 38.1 0)
+    (effects (font (size 1.27 1.27)) (justify left))
+  )
+  (hierarchical_label "CEN" (shape input) (at 17.78 68.58 180)
+    (effects (font (size 1.27 1.27)) (justify right))
+  )
+  (hierarchical_label "~{RQ}{slash}~{GT1}" (shape input) (at 184.15 96.52 0)
     (effects (font (size 1.27 1.27)) (justify left))
   )
@@
     (pin "1")
   )
+  (symbol (lib_id "Device:Buzzer") (at 96.52 21.59 90) (unit 1)
+    (in_bom yes) (on_board yes) (fields_autoplaced)
+    (property "Reference" "BZ1" (id 0) (at 100.33 19.5579 90)
+      (effects (font (size 1.27 1.27)) (justify right))
+    )
+    (property "Value" "Buzzer" (id 1) (at 100.33 22.0979 90)
+      (effects (font (size 1.27 1.27)) (justify right))
+    )
+    (property "Footprint" "Buzzer_Beeper:Buzzer_12x9.5RM7.6" (id 2) (at 93.98 22.225 90)
+      (effects (font (size 1.27 1.27)) hide)
+    )
+    (property "Datasheet" "~" (id 3) (at 93.98 22.225 90)
+      (effects (font (size 1.27 1.27)) hide)
+    )
+    (pin "1")
+    (pin "2")
+  )
   (symbol (lib_id "logo:LOGO") (at 288.29 262.89 0) (unit 1)
     (in_bom yes) (on_board yes) (fields_autoplaced)
@@
     (pin "9")
   )
+  (symbol (lib_id "power:GND") (at 99.06 29.21 0) (unit 1)
+    (in_bom yes) (on_board yes) (fields_autoplaced)
+    (property "Reference" "#PWR0109" (id 0) (at 99.06 35.56 0)
+      (effects (font (size 1.27 1.27)) hide)
+    )
+    (property "Value" "GND" (id 1) (at 99.06 34.29 0))
+    (property "Footprint" "" (id 2) (at 99.06 29.21 0)
+      (effects (font (size 1.27 1.27)) hide)
+    )
+    (property "Datasheet" "" (id 3) (at 99.06 29.21 0)
+      (effects (font (size 1.27 1.27)) hide)
+    )
+    (pin "1")
+  )
   (symbol (lib_id "power:GND") (at 151.13 34.29 0) (unit 1)
     (in_bom yes) (on_board yes) (fields_autoplaced)
@@
       (reference "#PWR0108") (unit 1) (value "GND") (footprint "")
     )
+    (path "/dc6ab99b-f697-4724-8513-d33fff819a5d"
+      (reference "#PWR0109") (unit 1) (value "GND") (footprint "")
+    )
+    (path "/95f4cd4e-0348-4031-904b-b4de132b066e"
+      (reference "BZ1") (unit 1) (value "Buzzer") (footprint "Buzzer_Beeper:Buzzer_12x9.5RM7.6")
+    )
     (path "/f22b9fda-18f5-4e76-a839-a6b0b67a7c59"
