File: 8088_pcb/kicad/ard8088.kicad_sch (KiCad schematic)
At the start: 6 parts, among them U1 8088_Max_Mode, U2 8288

Commit message: update kicad project
Parts:
- added D1, D2: LED, LED_SMD:LED_0805_2012Metric_Pad1.15x1.40mm_HandSolder, symbol Device:LED
- added R1, R2: R, Resistor_SMD:R_0805_2012Metric_Pad1.20x1.40mm_HandSolder, symbol Device:R
Connections:
- net +5V: now also XA1.3V3 (3.3V), R2.1; no longer XA1.5V1 (5V)
- net ALE: now also R1.1
- net GND: now also XA1. (S3), D1.1 (K), D2.1 (K)
- net +5Vactual: now reaches XA1.5V3 (5V)
- net +5Vactual: now also XA1. (S3), XA1.5V4 (5V)
- net ~{BHE}: now reaches XA1.D17 (D17_RX2)
- net ~{BHE}: now also U1.34 (HIGH)
- net ser0: now reaches XA1.D18 (D18_TX1)
- net ser0: now also XA1. (S3)
- net ser1: now reaches XA1.D19 (D19_RX1)
- net ser1: now also XA1. (S3)
- new net: D1.2 (A), R1.2
- new net: D2.2 (A), R2.2
- no-connect marks 12 -> 14
Other:
- title: Ard8088 -> Arduino8088
